File: BlueHand_mids/midsv3.kicad_pcb (KiCad board)
At the start: 2 copper layers, 10 parts

Commit message: added new mid plate - helps not confuse the laser cutter not mess things up and skip things
Parts:
- removed H1, H10, H2, H3, H4, H5, H6, H7, H8, H9: MountingHole_Pad, MountingHole:MountingHole_2.2mm_M2_Pad_TopBottom
Other:
- net class Default removed
- board text added: "PACKAGE IN SMALL GROUPS FOR BETTER SHIPPING OF FRAGILE PARTS"
- board text added: "THIS EXTRA MATERIAL IS NOT NEEDED"
- board text added: "THIS FILE MAKES 2 PARTS"
- board text added: "THIS SPACE IS EMPTY"
